Commit message: Work complete. US Closed.

File: urdf/scout.urdf (robot description, URDF)
Before this commit: robot scout, 5 links, 4 joints
Links:
- added link boom; visual mesh filename=package://icarus_rover_v2/meshes/365001.stl scale=.001 .001 .001
- added link bucket; visual mesh filename=package://icarus_rover_v2/meshes/365000.stl scale=.001 .001 .001
- link base_link: geometry visual mesh filename=package://icarus_rover_v2/meshes/base.stl scale=.001 .001 .001
Joints:
- added joint joint_boom_rotate: type continuous, parent base_link, child boom, origin xyz=.184 0 .112 rpy=0 0 0, axis 0 1 0
- added joint joint_bucket_rotate: type continuous, parent boom, child bucket, origin xyz=.172 0 -.0413 rpy=0 0 0, axis 0 1 0
